Commit message: Rainbow: tight conservative spheres against the master (197 -> 1070), every collidable self pair, clustered kernel
The four Rainbow kernels (rainbow/rainbowl, rainbowcam/rainbowcaml: 1070 /
1134 spheres) regenerated from the cricket inputs of the same name
(resources/rainbow, cricket branch rainbow-refit-1004):

- Every link's spheres cover the hull of its collision geometry in QAA's
  rainbow_seiji.urdf / rainbowcam_seiji.urdf within 6-20 mm per link
  (fingers 6, hand 8, wheels 10, base 15; 1 mm radius pad), verified on
  dense independent samples. Base, wheel and lidar spheres stay above
  z = 0.5 mm and cover the hulls from z = 12 mm up (the PO floor body).
  The old set left up to 47 mm of the hulls uncovered (base, torso_5) and
  protruded up to 75 mm (wheels) and 155 mm (head).
- The lidar (a box on the base, not modelled before) is covered.
- The head camera mount is covered over the head's whole pan/tilt range:
  VAMP has no head DOF, and a cover at tilt 0 alone missed 30-50% of the
  arm-vs-camera hits at the head's real tilts.
- torso_2's limits follow the master ([-140, +80] deg; was [-142, +90]).
- SRDF: every pair that can collide is checked (421 of 630; 478 of 703
  with the wrist cameras). Disabled: the derived exclusions (qaa
  robot_description), pairs fixed in VAMP's model, pairs whose hulls never
  touch within the limits (random census of 240k confs + distance
  minimisation), and torso_5 vs arm_1 (hulls 5 mm apart at the stow conf).
  The old SRDF checked 86 pairs (distal arm x torso), no arm vs head/camera,
  base, other arm or own arm.
- The kernel screens each link pair through sphere clusters (an anchor
  sphere + constant radius) before the sphere pairs, and runs the sphere
  tests out of line: the flat cricket template would need 394k unrolled
  sphere-pair tests per function.

Against the master's hulls in a table scene (20k confs): false-valid
953 -> 0; kernel verdicts equal a direct sphere computation on all 20k
(and the attachment path on 6k). validate() 3.1 -> 8.7 us on valid confs.

Co-Authored-By: Claude Opus 5.5 <noreply@anthropic.com>

File: resources/rainbow/rainbow_spherized.urdf (robot description, URDF)
Before this commit: robot RB_Y1_V1.0.1, 40 links, 39 joints
Links:
- added link lidar_mid360; collision sphere radius=0.009537; collision sphere radius=0.009611
- added link tcp_left
- added link tcp_right
- link FT_sensor_L: geometry collision sphere radius=0.007295; collision sphere radius=0.015905
- link FT_sensor_R: geometry collision sphere radius=0.009062; collision sphere radius=0.017838
- link base: geometry collision sphere radius=0.010238; collision sphere radius=0.019799
- link ee_finger_l1: geometry collision sphere radius=0.009736; collision sphere radius=0.010047
- link ee_finger_l2: geometry collision sphere radius=0.009736; collision sphere radius=0.010047
- link ee_finger_r1: geometry collision sphere radius=0.009736; collision sphere radius=0.010047
- link ee_finger_r2: geometry collision sphere radius=0.009736; collision sphere radius=0.010047
- link ee_left: geometry collision sphere radius=0.006781; collision sphere radius=0.008223
- link ee_right: geometry collision sphere radius=0.006781; collision sphere radius=0.008223
- link link_head_0: geometry collision sphere radius=0.018214; collision sphere radius=0.018874
- link link_head_1: geometry collision sphere radius=0.030197; collision sphere radius=0.036620
- link link_head_2: geometry collision sphere radius=0.013767; collision sphere radius=0.020647
- link link_left_arm_0: geometry collision sphere radius=0.016096; collision sphere radius=0.026753
- link link_left_arm_1: geometry collision sphere radius=0.021128; collision sphere radius=0.021433
- link link_left_arm_2: geometry collision sphere radius=0.013206; collision sphere radius=0.015616
- link link_left_arm_3: geometry collision sphere radius=0.012527; collision sphere radius=0.017003
- link link_left_arm_4: geometry collision sphere radius=0.012398; collision sphere radius=0.019829
- link link_left_arm_5: geometry collision sphere radius=0.012333; collision sphere radius=0.014731
- link link_left_arm_6: geometry collision sphere radius=0.017306; collision sphere radius=0.017942
- link link_right_arm_0: geometry collision sphere radius=0.030422; collision sphere radius=0.030815
- link link_right_arm_1: geometry collision sphere radius=0.021164; collision sphere radius=0.021439
- link link_right_arm_2: geometry collision sphere radius=0.014534; collision sphere radius=0.017995
- link link_right_arm_3: geometry collision sphere radius=0.017024; collision sphere radius=0.023816
- link link_right_arm_4: geometry collision sphere radius=0.010469; collision sphere radius=0.010515
- link link_right_arm_5: geometry collision sphere radius=0.011540; collision sphere radius=0.011796
- link link_right_arm_6: geometry collision sphere radius=0.011703; collision sphere radius=0.013588
- link link_torso_0: geometry collision sphere radius=0.039300; collision sphere radius=0.042782
- link link_torso_1: geometry collision sphere radius=0.034444; collision sphere radius=0.035390
- link link_torso_2: geometry collision sphere radius=0.023369; collision sphere radius=0.025093
- link link_torso_3: geometry collision sphere radius=0.024259; collision sphere radius=0.042680
- link link_torso_4: geometry collision sphere radius=0.017617; collision sphere radius=0.018456
- link link_torso_5: geometry collision sphere radius=0.014299; collision sphere radius=0.015322
- link rby1_camera_mount: geometry collision sphere radius=0.072041; collision sphere radius=0.085635
- link wheel_l: geometry collision sphere radius=0.013979; collision sphere radius=0.017978
- link wheel_r: geometry collision sphere radius=0.013979; collision sphere radius=0.017978
Joints:
- added joint lidar_mid360_mount: type fixed, parent base, child lidar_mid360, origin xyz=0.25 0 0.2 rpy=0 0 0
- added joint tcp_joint_left: type fixed, parent grasp_frame_left, child tcp_left, origin xyz=0 0 0 rpy=-3.14159265358979 0 1.57079632679490
- added joint tcp_joint_right: type fixed, parent grasp_frame_right, child tcp_right, origin xyz=0 0 0 rpy=-3.14159265358979 0 1.57079632679490
- joint torso_2: limit lower=-2.478367 upper=1.570796327 effort=270.0 velocity=2.09439510 -> lower=-2.4434609528 upper=1.3962634016 effort=270.0 velocity=2.09439510

File: resources/rainbow/rainbowcam_spherized.urdf (robot description, URDF)
Before this commit: robot RB_Y1_V1.0.1, 42 links, 41 joints
Links:
- added link lidar_mid360; collision sphere radius=0.009537; collision sphere radius=0.009611
- added link tcp_left
- added link tcp_right
- link FT_sensor_L: geometry collision sphere radius=0.007295; collision sphere radius=0.015905
- link FT_sensor_R: geometry collision sphere radius=0.009062; collision sphere radius=0.017838
- link base: geometry collision sphere radius=0.010238; collision sphere radius=0.019799
- link ee_finger_l1: geometry collision sphere radius=0.009736; collision sphere radius=0.010047
- link ee_finger_l2: geometry collision sphere radius=0.009736; collision sphere radius=0.010047
- link ee_finger_r1: geometry collision sphere radius=0.009736; collision sphere radius=0.010047
- link ee_finger_r2: geometry collision sphere radius=0.009736; collision sphere radius=0.010047
- link ee_left: geometry collision sphere radius=0.006781; collision sphere radius=0.008223
- link ee_right: geometry collision sphere radius=0.006781; collision sphere radius=0.008223
- link link_head_0: geometry collision sphere radius=0.018214; collision sphere radius=0.018874
- link link_head_1: geometry collision sphere radius=0.030197; collision sphere radius=0.036620
- link link_head_2: geometry collision sphere radius=0.013767; collision sphere radius=0.020647
- link link_left_arm_0: geometry collision sphere radius=0.016096; collision sphere radius=0.026753
- link link_left_arm_1: geometry collision sphere radius=0.021128; collision sphere radius=0.021433
- link link_left_arm_2: geometry collision sphere radius=0.013206; collision sphere radius=0.015616
- link link_left_arm_3: geometry collision sphere radius=0.012527; collision sphere radius=0.017003
- link link_left_arm_4: geometry collision sphere radius=0.012398; collision sphere radius=0.019829
- link link_left_arm_5: geometry collision sphere radius=0.012333; collision sphere radius=0.014731
- link link_left_arm_6: geometry collision sphere radius=0.017306; collision sphere radius=0.017942
- link link_left_arm_camera: geometry collision sphere radius=0.005623; collision sphere radius=0.007580
- link link_right_arm_0: geometry collision sphere radius=0.030422; collision sphere radius=0.030815
- link link_right_arm_1: geometry collision sphere radius=0.021164; collision sphere radius=0.021439
- link link_right_arm_2: geometry collision sphere radius=0.014534; collision sphere radius=0.017995
- link link_right_arm_3: geometry collision sphere radius=0.017024; collision sphere radius=0.023816
- link link_right_arm_4: geometry collision sphere radius=0.010469; collision sphere radius=0.010515
- link link_right_arm_5: geometry collision sphere radius=0.011540; collision sphere radius=0.011796
- link link_right_arm_6: geometry collision sphere radius=0.011703; collision sphere radius=0.013588
- link link_right_arm_camera: geometry collision sphere radius=0.007711; collision sphere radius=0.009301
- link link_torso_0: geometry collision sphere radius=0.039300; collision sphere radius=0.042782
- link link_torso_1: geometry collision sphere radius=0.034444; collision sphere radius=0.035390
- link link_torso_2: geometry collision sphere radius=0.023369; collision sphere radius=0.025093
- link link_torso_3: geometry collision sphere radius=0.024259; collision sphere radius=0.042680
- link link_torso_4: geometry collision sphere radius=0.017617; collision sphere radius=0.018456
- link link_torso_5: geometry collision sphere radius=0.014299; collision sphere radius=0.015322
- link rby1_camera_mount: geometry collision sphere radius=0.072041; collision sphere radius=0.085635
- link wheel_l: geometry collision sphere radius=0.013979; collision sphere radius=0.017978
- link wheel_r: geometry collision sphere radius=0.013979; collision sphere radius=0.017978
Joints:
- added joint lidar_mid360_mount: type fixed, parent base, child lidar_mid360, origin xyz=0.25 0 0.2 rpy=0 0 0
- added joint tcp_joint_left: type fixed, parent grasp_frame_left, child tcp_left, origin xyz=0 0 0 rpy=-3.14159265358979 0 1.57079632679490
- added joint tcp_joint_right: type fixed, parent grasp_frame_right, child tcp_right, origin xyz=0 0 0 rpy=-3.14159265358979 0 1.57079632679490
- joint torso_2: limit lower=-2.478367 upper=1.570796327 effort=270.0 velocity=2.09439510 -> lower=-2.4434609528 upper=1.3962634016 effort=270.0 velocity=2.09439510
